Commit message: Added Gazebo

File: navigation-c/models/robot_configuration.urdf (robot description, URDF)
Before this commit: robot differential_robot, 2 links, 1 joints
Links:
- added link imu_link; collision box size=0.1 0.1 0.1; visual box size=0.1 0.1 0.1
- link base_link: geometry collision box size=${base_length} ${base_width} ${base_height}; visual box size=${base_length} ${base_width} ${base_height}
Joints:
- added joint imu_joint: type fixed, parent base_link, child imu_link, origin xyz=0 0 0.01

Commit message: lidar sensor

File: navigation-c/models/robot_configuration.urdf (robot description, URDF)
Before this commit: robot differential_robot, 3 links, 2 joints
Links:
- added link camera_depth_frame
- added link camera_link, mass 0.035; collision box size=0.015 0.130 0.022; visual box size=0.015 0.130 0.022
- added link lidar_link, mass 0.125; collision cylinder length=0.055 radius=0.0508; visual cylinder length=0.055 radius=0.0508
Joints:
- added joint camera_depth_joint: type fixed, parent camera_link, child camera_depth_frame, origin xyz=0 0 0 rpy=${-pi/2} 0 ${-pi/2}
- added joint camera_joint: type fixed, parent base_link, child camera_link, origin xyz=0.215 0 0.05 rpy=0 0 0
- added joint lidar_joint: type fixed, parent base_link, child lidar_link, origin xyz=0 0 0.26 rpy=0 0 0

Commit message: added Lidar

File: navigation-c/models/robot_configuration.urdf (robot description, URDF)
Before this commit: robot differential_robot, 3 links, 2 joints
Links:
- link imu_link: geometry visual box size=0.1 0.1 0.1

Commit message: moved camera

File: navigation-c/models/robot_configuration.urdf (robot description, URDF)
Before this commit: robot differential_robot, 6 links, 5 joints
Joints:
- joint camera_joint: origin xyz=0.215 0 0.05 rpy=0 0 0 -> xyz=0.50 0 0.05 rpy=0 0 0

Commit message: Moved LIDAR to Front

File: navigation-c/models/robot_configuration.urdf (robot description, URDF)
Before this commit: robot differential_robot, 6 links, 5 joints
Joints:
- joint lidar_joint: origin xyz=0 0 0.26 rpy=0 0 0 -> xyz=0.5 0 0.26 rpy=0 0 0
