Commit message: Robot model, wheels square

File: src/description/sam_bot_description_tutorial.urdf (robot description, URDF)
Before this commit: robot sam_bot, 6 links, 5 joints
Joints:
- joint camera_joint: origin xyz=0.215 0 0.05 rpy=0 0 0 -> xyz=0.7575 0 0.05 rpy=0 0 0
- joint lidar_joint: origin xyz=0 0 0.12 rpy=0 0 0 -> xyz=0 0 0.4025 rpy=0 0 0
